File: dac_shield.sch (KiCad schematic (older format))
At the start: 15 parts

Commit message: some changes
Parts:
- removed U?: MCP4921, symbol MCP4921
- gave numbers to parts that had none: 13
Connections:
- net labels added: MCP4921
Changed lines of the file:
@@
 LIBS:mcp4921
 LIBS:custom_parts
+LIBS:dac_shield-cache
 EELAYER 27 0
 EELAYER END
@@
 Sheet 1 1
 Title "Power DAC Shield"
-Date "14 jul 2013"
+Date "15 jul 2013"
 Rev ""
 Comp "Visgence Inc."
@@
 $EndDescr
 $Comp
-L ARDUINO_SHIELD SHIELD?
+L ARDUINO_SHIELD SHIELD1
 U 1 1 51E2FC01
 P 2450 2150
-F 0 "SHIELD?" H 2100 3100 60  0000 C CNN
+F 0 "SHIELD1" H 2100 3100 60  0000 C CNN
 F 1 "ARDUINO_SHIELD" H 2500 1200 60  0000 C CNN
 F 2 "" H 2450 2150 60  0000 C CNN
@@
 $EndComp
 $Comp
-L MCP4921 U?
+L MCP4921 #U01
 U 1 1 51E2FDD6
 P 5750 2300
-F 0 "U?" H 5750 2650 60  0000 C CNN
+F 0 "#U01" H 5750 2650 60  0000 C CNN
 F 1 "MCP4921" H 5550 1850 60  0000 C CNN
 F 2 "" H 5750 2300 60  0000 C CNN
@@
 	5150 2550 5350 2550
 $Comp
-L CONN_4X2 P?
+L CONN_4X2 P1
 U 1 1 51E3006B
 P 4200 2000
-F 0 "P?" H 4200 2250 50  0000 C CNN
+F 0 "P1" H 4200 2250 50  0000 C CNN
 F 1 "SLAVE_SEL" V 4200 2000 40  0000 C CNN
 F 2 "" H 4200 2000 60  0000 C CNN
@@
 Connection ~ 4600 1950
 $Comp
-L +5V #PWR?
+L +5V #PWR02
 U 1 1 51E300D3
 P 1200 1800
-F 0 "#PWR?" H 1200 1890 20  0001 C CNN
+F 0 "#PWR02" H 1200 1890 20  0001 C CNN
 F 1 "+5V" H 1200 1890 30  0000 C CNN
 F 2 "" H 1200 1800 60  0000 C CNN
@@
 $EndComp
 $Comp
-L +5V #PWR?
+L +5V #PWR03
 U 1 1 51E300EF
 P 5200 1950
-F 0 "#PWR?" H 5200 2040 20  0001 C CNN
+F 0 "#PWR03" H 5200 2040 20  0001 C CNN
 F 1 "+5V" H 5200 2040 30  0000 C CNN
 F 2 "" H 5200 1950 60  0000 C CNN
@@
 	5200 2100 5200 1950
 $Comp
-L GND #PWR?
+L GND #PWR04
 U 1 1 51E30124
 P 3900 1550
-F 0 "#PWR?" H 3900 1550 30  0001 C CNN
+F 0 "#PWR04" H 3900 1550 30  0001 C CNN
 F 1 "GND" H 3900 1480 30  0001 C CNN
 F 2 "" H 3900 1550 60  0000 C CNN
@@
 	3900 1450 3900 1550
 $Comp
-L GND #PWR?
+L GND #PWR05
 U 1 1 51E3017A
 P 1150 2200
-F 0 "#PWR?" H 1150 2200 30  0001 C CNN
+F 0 "#PWR05" H 1150 2200 30  0001 C CNN
 F 1 "GND" H 1150 2130 30  0001 C CNN
 F 2 "" H 1150 2200 60  0000 C CNN
@@
 $EndComp
 $Comp
-L GND #PWR?
+L GND #PWR06
 U 1 1 51E30180
 P 6350 2300
-F 0 "#PWR?" H 6350 2300 30  0001 C CNN
+F 0 "#PWR06" H 6350 2300 30  0001 C CNN
 F 1 "GND" H 6350 2230 30  0001 C CNN
 F 2 "" H 6350 2300 60  0000 C CNN
@@
 	6350 2250 6350 2300
 $Comp
-L TCA0372 U?
+L TCA0372 U2
 U 2 1 51E30546
 P 6000 4550
-F 0 "U?" H 6000 4700 60  0000 L CNN
+F 0 "U2" H 6000 4700 60  0000 L CNN
 F 1 "TCA0372" H 6200 4350 60  0000 C CNN
 F 2 "" H 6000 4550 60  0000 C CNN
@@
 $EndComp
 $Comp
-L TCA0372 U?
+L TCA0372 U2
 U 1 1 51E30553
 P 4700 4550
-F 0 "U?" H 4700 4700 60  0000 L CNN
+F 0 "U2" H 4700 4700 60  0000 L CNN
 F 1 "TCA0372" H 4900 4350 60  0000 C CNN
 F 2 "" H 4700 4550 60  0000 C CNN
@@
 	5350 4450 5650 4450
 $Comp
-L R R?
+L R R4
 U 1 1 51E30590
 P 4650 5150
-F 0 "R?" V 4730 5150 40  0000 C CNN
+F 0 "R4" V 4730 5150 40  0000 C CNN
 F 1 "10k" V 4657 5151 40  0000 C CNN
 F 2 "~" V 4580 5150 30  0000 C CNN
@@
 	4350 5150 4350 4650
 $Comp
-L POT RV?
+L POT RV1
 U 1 1 51E30660
 P 5650 5200
-F 0 "RV?" H 5650 5100 50  0000 C CNN
+F 0 "RV1" H 5650 5100 50  0000 C CNN
 F 1 "10k" H 5650 5200 50  0000 C CNN
 F 2 "~" H 5650 5200 60  0000 C CNN
@@
 $EndComp
 $Comp
-L VSS #PWR?
+L VSS #PWR07
 U 1 1 51E3066F
 P 5900 4900
-F 0 "#PWR?" H 5900 4900 30  0001 C CNN
+F 0 "#PWR07" H 5900 4900 30  0001 C CNN
 F 1 "VSS" H 5900 4830 30  0000 C CNN
 F 2 "" H 5900 4900 60  0000 C CNN
@@
 $EndComp
 $Comp
-L VDD #PWR?
+L VDD #PWR08
 U 1 1 51E3067E
 P 5900 4150
-F 0 "#PWR?" H 5900 4250 30  0001 C CNN
+F 0 "#PWR08" H 5900 4250 30  0001 C CNN
 F 1 "VDD" H 5900 4260 30  0000 C CNN
 F 2 "" H 5900 4150 60  0000 C CNN
@@
 $EndComp
 $Comp
-L VDD #PWR?
+L VDD #PWR09
 U 1 1 51E3068B
 P 4600 4150
-F 0 "#PWR?" H 4600 4250 30  0001 C CNN
+F 0 "#PWR09" H 4600 4250 30  0001 C CNN
 F 1 "VDD" H 4600 4260 30  0000 C CNN
 F 2 "" H 4600 4150 60  0000 C CNN
@@
 $EndComp
 $Comp
-L VSS #PWR?
+L VSS #PWR010
 U 1 1 51E30691
 P 4600 4900
-F 0 "#PWR?" H 4600 4900 30  0001 C CNN
+F 0 "#PWR010" H 4600 4900 30  0001 C CNN
 F 1 "VSS" H 4600 4830 30  0000 C CNN
 F 2 "" H 4600 4900 60  0000 C CNN
@@
 	5650 5050 5650 4650
 $Comp
-L R R?
+L R R6
 U 1 1 51E30757
 P 6300 5200
-F 0 "R?" V 6380 5200 40  0000 C CNN
+F 0 "R6" V 6380 5200 40  0000 C CNN
 F 1 "33k" V 6307 5201 40  0000 C CNN
 F 2 "~" V 6230 5200 30  0000 C CNN
@@
 	6350 4550 7450 4550
 $Comp
-L R R?
+L R R5
 U 1 1 51E307BD
 P 5300 5550
-F 0 "R?" V 5380 5550 40  0000 C CNN
+F 0 "R5" V 5380 5550 40  0000 C CNN
 F 1 "12k" V 5307 5551 40  0000 C CNN
 F 2 "~" V 5230 5550 30  0000 C CNN
@@
 	5300 5200 5400 5200
 $Comp
-L GND #PWR?
+L GND #PWR011
 U 1 1 51E307ED
 P 5300 5950
-F 0 "#PWR?" H 5300 5950 30  0001 C CNN
+F 0 "#PWR011" H 5300 5950 30  0001 C CNN
 F 1 "GND" H 5300 5880 30  0001 C CNN
 F 2 "" H 5300 5950 60  0000 C CNN
@@
 	5300 5800 5300 5950
 $Comp
-L R R?
+L R R3
 U 1 1 51E3081F
 P 3900 4650
-F 0 "R?" V 3980 4650 40  0000 C CNN
+F 0 "R3" V 3980 4650 40  0000 C CNN
 F 1 "10k" V 3907 4651 40  0000 C CNN
 F 2 "~" V 3830 4650 30  0000 C CNN
@@
 DAC_OUT
 $Comp
-L LM741 U?
+L LM741 U1
 U 1 1 51E30A12
 P 2100 4650
-F 0 "U?" H 2250 4800 60  0000 C CNN
+F 0 "U1" H 2250 4800 60  0000 C CNN
 F 1 "LM741" H 2250 4900 60  0000 C CNN
 F 2 "" H 2100 4650 60  0000 C CNN
@@
 	1600 5200 1600 4750
 $Comp
-L VSS #PWR?
+L VSS #PWR012
 U 1 1 51E30A90
 P 2000 5100
-F 0 "#PWR?" H 2000 5100 30  0001 C CNN
+F 0 "#PWR012" H 2000 5100 30  0001 C CNN
 F 1 "VSS" H 2000 5030 30  0000 C CNN
 F 2 "" H 2000 5100 60  0000 C CNN
@@
 	2000 5050 2000 5100
 $Comp
-L VDD #PWR?
+L VDD #PWR013
 U 1 1 51E30AC8
 P 2000 4150
-F 0 "#PWR?" H 2000 4250 30  0001 C CNN
+F 0 "#PWR013" H 2000 4250 30  0001 C CNN
 F 1 "VDD" H 2000 4260 30  0000 C CNN
 F 2 "" H 2000 4150 60  0000 C CNN
@@
 	2000 4150 2000 4250
 $Comp
-L R R?
+L R R1
 U 1 1 51E30B0D
 P 1400 4300
-F 0 "R?" V 1480 4300 40  0000 C CNN
+F 0 "R1" V 1480 4300 40  0000 C CNN
 F 1 "22k" V 1407 4301 40  0000 C CNN
 F 2 "~" V 1330 4300 30  0000 C CNN
@@
 $EndComp
 $Comp
-L VDD #PWR?
+L VDD #PWR014
 U 1 1 51E30B13
 P 1400 3950
-F 0 "#PWR?" H 1400 4050 30  0001 C CNN
+F 0 "#PWR014" H 1400 4050 30  0001 C CNN
 F 1 "VDD" H 1400 4060 30  0000 C CNN
 F 2 "" H 1400 3950 60  0000 C CNN
@@
 $EndComp
 $Comp
-L R R?
+L R R2
 U 1 1 51E30B19
 P 1400 4900
-F 0 "R?" V 1480 4900 40  0000 C CNN
+F 0 "R2" V 1480 4900 40  0000 C CNN
 F 1 "10k" V 1407 4901 40  0000 C CNN
 F 2 "~" V 1330 4900 30  0000 C CNN
@@
 $EndComp
 $Comp
-L GND #PWR?
+L GND #PWR015
 U 1 1 51E30B25
 P 1400 5250
-F 0 "#PWR?" H 1400 5250 30  0001 C CNN
+F 0 "#PWR015" H 1400 5250 30  0001 C CNN
 F 1 "GND" H 1400 5180 30  0001 C CNN
 F 2 "" H 1400 5250 60  0000 C CNN
@@
 	1200 1950 1200 1800
 $Comp
-L CONN_3 K?
+L CONN_3 K1
 U 1 1 51E30D77
 P 8100 3000
-F 0 "K?" V 8050 3000 50  0000 C CNN
+F 0 "K1" V 8050 3000 50  0000 C CNN
 F 1 "CONN_3" V 8150 3000 40  0000 C CNN
 F 2 "" H 8100 3000 60  0000 C CNN
@@
 $EndComp
 $Comp
-L VDD #PWR?
+L VDD #PWR016
 U 1 1 51E30D84
 P 7500 2800
-F 0 "#PWR?" H 7500 2900 30  0001 C CNN
+F 0 "#PWR016" H 7500 2900 30  0001 C CNN
 F 1 "VDD" H 7500 2910 30  0000 C CNN
 F 2 "" H 7500 2800 60  0000 C CNN
@@
 	7500 2900 7500 2800
 $Comp
-L VSS #PWR?
+L VSS #PWR017
 U 1 1 51E30DC8
 P 7500 3250
-F 0 "#PWR?" H 7500 3250 30  0001 C CNN
+F 0 "#PWR017" H 7500 3250 30  0001 C CNN
 F 1 "VSS" H 7500 3180 30  0000 C CNN
 F 2 "" H 7500 3250 60  0000 C CNN
@@
 	7500 3100 7500 3250
 $Comp
-L GND #PWR?
+L GND #PWR018
 U 1 1 51E30E0E
 P 7350 3050
-F 0 "#PWR?" H 7350 3050 30  0001 C CNN
+F 0 "#PWR018" H 7350 3050 30  0001 C CNN
 F 1 "GND" H 7350 2980 30  0001 C CNN
 F 2 "" H 7350 3050 60  0000 C CNN
@@
 	7350 3000 7750 3000
 $Comp
-L CONN_2 P?
+L CONN_2 P2
 U 1 1 51E30EA9
 P 7800 4650
-F 0 "P?" V 7750 4650 40  0000 C CNN
+F 0 "P2" V 7750 4650 40  0000 C CNN
 F 1 "CONN_2" V 7850 4650 40  0000 C CNN
 F 2 "" H 7800 4650 60  0000 C CNN
@@
 Connection ~ 6550 4550
 $Comp
-L GND #PWR?
+L GND #PWR019
 U 1 1 51E30EF3
 P 7300 4850
-F 0 "#PWR?" H 7300 4850 30  0001 C CNN
+F 0 "#PWR019" H 7300 4850 30  0001 C CNN
 F 1 "GND" H 7300 4780 30  0001 C CNN
 F 2 "" H 7300 4850 60  0000 C CNN

Commit message: Added leds and caps
Parts:
- added C1: 100n, ~, symbol C
- added C2: 47u, ~, symbol C
- added C3, C4: 1u, ~, symbol C
- added D1: PWR, ~, symbol LED
- added D2: POS, ~, symbol LED
- added D3: NEG, ~, symbol LED
- added R7, R8, R9: 1k, ~, symbol R
Connections:
- wire segments 64 -> 89

Commit message: Added logos, moved parts around
Parts:
- removed K1: CONN_3, symbol CONN_3
- removed P2: CONN_2, symbol CONN_2
- added P1: V+, symbol CONN_1
- added P2, P5: GND, symbol CONN_1
- added P3: V-, symbol CONN_1
- added P4: Out, symbol CONN_1
- renumbered P1 to JP1
Changed lines of the file:
@@
 $EndComp
 $Comp
-L MCP4921 #U01
+L MCP4921 #U1
 U 1 1 51E2FDD6
 P 5750 2300
-F 0 "#U01" H 5750 2650 60  0001 C CNN
+F 0 "#U1" H 5750 2650 60  0001 C CNN
 F 1 "MCP4921" H 5550 1850 60  0000 C CNN
 F 2 "" H 5750 2300 60  0000 C CNN
@@
 	5150 2550 5350 2550
 $Comp
-L CONN_4X2 P1
+L CONN_4X2 JP1
 U 1 1 51E3006B
 P 4200 2000
-F 0 "P1" H 4200 2250 50  0000 C CNN
+F 0 "JP1" H 4200 2250 50  0000 C CNN
 F 1 "SLAVE_SEL" V 4200 2000 40  0000 C CNN
 F 2 "" H 4200 2000 60  0000 C CNN
@@
 Connection ~ 4600 1950
 $Comp
-L +5V #PWR02
+L +5V #PWR2
 U 1 1 51E300D3
 P 1200 1800
-F 0 "#PWR02" H 1200 1890 20  0001 C CNN
+F 0 "#PWR2" H 1200 1890 20  0001 C CNN
 F 1 "+5V" H 1200 1890 30  0000 C CNN
 F 2 "" H 1200 1800 60  0000 C CNN
@@
 $EndComp
 $Comp
-L +5V #PWR03
+L +5V #PWR11
 U 1 1 51E300EF
 P 5200 1950
-F 0 "#PWR03" H 5200 2040 20  0001 C CNN
+F 0 "#PWR11" H 5200 2040 20  0001 C CNN
 F 1 "+5V" H 5200 2040 30  0000 C CNN
 F 2 "" H 5200 1950 60  0000 C CNN
@@
 	5200 2100 5200 1950
 $Comp
-L GND #PWR04
+L GND #PWR7
 U 1 1 51E30124
 P 3900 1550
-F 0 "#PWR04" H 3900 1550 30  0001 C CNN
+F 0 "#PWR7" H 3900 1550 30  0001 C CNN
 F 1 "GND" H 3900 1480 30  0001 C CNN
 F 2 "" H 3900 1550 60  0000 C CNN
@@
 	3900 1450 3900 1550
 $Comp
-L GND #PWR05
+L GND #PWR1
 U 1 1 51E3017A
 P 1150 2200
-F 0 "#PWR05" H 1150 2200 30  0001 C CNN
+F 0 "#PWR1" H 1150 2200 30  0001 C CNN
 F 1 "GND" H 1150 2130 30  0001 C CNN
 F 2 "" H 1150 2200 60  0000 C CNN
@@
 $EndComp
 $Comp
-L GND #PWR06
+L GND #PWR15
 U 1 1 51E30180
 P 6350 2300
-F 0 "#PWR06" H 6350 2300 30  0001 C CNN
+F 0 "#PWR15" H 6350 2300 30  0001 C CNN
 F 1 "GND" H 6350 2230 30  0001 C CNN
 F 2 "" H 6350 2300 60  0000 C CNN
@@
 $EndComp
 $Comp
-L VSS #PWR07
+L VSS #PWR14
 U 1 1 51E3066F
 P 5900 4900
-F 0 "#PWR07" H 5900 4900 30  0001 C CNN
+F 0 "#PWR14" H 5900 4900 30  0001 C CNN
 F 1 "VSS" H 5900 4830 30  0000 C CNN
 F 2 "" H 5900 4900 60  0000 C CNN
@@
 $EndComp
 $Comp
-L VDD #PWR08
+L VDD #PWR13
 U 1 1 51E3067E
 P 5900 4150
-F 0 "#PWR08" H 5900 4250 30  0001 C CNN
+F 0 "#PWR13" H 5900 4250 30  0001 C CNN
 F 1 "VDD" H 5900 4260 30  0000 C CNN
 F 2 "" H 5900 4150 60  0000 C CNN
@@
 $EndComp
 $Comp
-L VDD #PWR09
+L VDD #PWR8
 U 1 1 51E3068B
 P 4600 4150
-F 0 "#PWR09" H 4600 4250 30  0001 C CNN
+F 0 "#PWR8" H 4600 4250 30  0001 C CNN
 F 1 "VDD" H 4600 4260 30  0000 C CNN
 F 2 "" H 4600 4150 60  0000 C CNN
@@
 $EndComp
 $Comp
-L VSS #PWR010
+L VSS #PWR9
 U 1 1 51E30691
 P 4600 4900
-F 0 "#PWR010" H 4600 4900 30  0001 C CNN
+F 0 "#PWR9" H 4600 4900 30  0001 C CNN
 F 1 "VSS" H 4600 4830 30  0000 C CNN
 F 2 "" H 4600 4900 60  0000 C CNN
@@
 	5300 5200 5400 5200
 $Comp
-L GND #PWR011
+L GND #PWR12
 U 1 1 51E307ED
 P 5300 5950
-F 0 "#PWR011" H 5300 5950 30  0001 C CNN
+F 0 "#PWR12" H 5300 5950 30  0001 C CNN
 F 1 "GND" H 5300 5880 30  0001 C CNN
 F 2 "" H 5300 5950 60  0000 C CNN
@@
 	1600 5200 1600 4750
 $Comp
-L VSS #PWR012
+L VSS #PWR6
 U 1 1 51E30A90
 P 2000 5100
-F 0 "#PWR012" H 2000 5100 30  0001 C CNN
+F 0 "#PWR6" H 2000 5100 30  0001 C CNN
 F 1 "VSS" H 2000 5030 30  0000 C CNN
 F 2 "" H 2000 5100 60  0000 C CNN
@@
 	2000 5050 2000 5100
 $Comp
-L VDD #PWR013
+L VDD #PWR5
 U 1 1 51E30AC8
 P 2000 4150
-F 0 "#PWR013" H 2000 4250 30  0001 C CNN
+F 0 "#PWR5" H 2000 4250 30  0001 C CNN
 F 1 "VDD" H 2000 4260 30  0000 C CNN
 F 2 "" H 2000 4150 60  0000 C CNN
@@
 $EndComp
 $Comp
-L VDD #PWR014
+L VDD #PWR3
 U 1 1 51E30B13
 P 1400 3950
-F 0 "#PWR014" H 1400 4050 30  0001 C CNN
+F 0 "#PWR3" H 1400 4050 30  0001 C CNN
 F 1 "VDD" H 1400 4060 30  0000 C CNN
 F 2 "" H 1400 3950 60  0000 C CNN
@@
 $EndComp
 $Comp
-L GND #PWR015
+L GND #PWR4
 U 1 1 51E30B25
 P 1400 5250
-F 0 "#PWR015" H 1400 5250 30  0001 C CNN
+F 0 "#PWR4" H 1400 5250 30  0001 C CNN
 F 1 "GND" H 1400 5180 30  0001 C CNN
 F 2 "" H 1400 5250 60  0000 C CNN
@@
 	1200 1950 1200 1800
 $Comp
-L CONN_3 K1
-U 1 1 51E30D77
-P 8100 3000
-F 0 "K1" V 8050 3000 50  0000 C CNN
-F 1 "CONN_3" V 8150 3000 40  0000 C CNN
-F 2 "" H 8100 3000 60  0000 C CNN
-F 3 "" H 8100 3000 60  0000 C CNN
-	1    8100 3000
-	1    0    0    -1
-$EndComp
-$Comp
-L VDD #PWR016
+L VDD #PWR18
 U 1 1 51E30D84
 P 7500 2800
-F 0 "#PWR016" H 7500 2900 30  0001 C CNN
+F 0 "#PWR18" H 7500 2900 30  0001 C CNN
 F 1 "VDD" H 7500 2910 30  0000 C CNN
 F 2 "" H 7500 2800 60  0000 C CNN
@@
 	7500 2900 7500 2800
 $Comp
-L VSS #PWR017
+L VSS #PWR19
 U 1 1 51E30DC8
 P 7500 3250
-F 0 "#PWR017" H 7500 3250 30  0001 C CNN
+F 0 "#PWR19" H 7500 3250 30  0001 C CNN
 F 1 "VSS" H 7500 3180 30  0000 C CNN
 F 2 "" H 7500 3250 60  0000 C CNN
@@
 	7500 3100 7500 3250
 $Comp
-L GND #PWR018
+L GND #PWR17
 U 1 1 51E30E0E
 P 7350 3050
-F 0 "#PWR018" H 7350 3050 30  0001 C CNN
+F 0 "#PWR17" H 7350 3050 30  0001 C CNN
 F 1 "GND" H 7350 2980 30  0001 C CNN
 F 2 "" H 7350 3050 60  0000 C CNN
@@
 Wire Wire Line
 	7350 3000 7750 3000
-$Comp
-L CONN_2 P2
-U 1 1 51E30EA9
-P 7800 4650
-F 0 "P2" V 7750 4650 40  0000 C CNN
-F 1 "CONN_2" V 7850 4650 40  0000 C CNN
-F 2 "" H 7800 4650 60  0000 C CNN
-F 3 "" H 7800 4650 60  0000 C CNN
-	1    7800 4650
-	1    0    0    -1
-$EndComp
 Connection ~ 6550 4550
 $Comp
-L GND #PWR019
+L GND #PWR16
 U 1 1 51E30EF3
 P 7300 4850
-F 0 "#PWR019" H 7300 4850 30  0001 C CNN
+F 0 "#PWR16" H 7300 4850 30  0001 C CNN
 F 1 "GND" H 7300 4780 30  0001 C CNN
 F 2 "" H 7300 4850 60  0000 C CNN
@@
 Connection ~ 5200 2100
 $Comp
-L GND #PWR020
+L GND #PWR10
 U 1 1 51E82617
 P 4750 3050
-F 0 "#PWR020" H 4750 3050 30  0001 C CNN
+F 0 "#PWR10" H 4750 3050 30  0001 C CNN
 F 1 "GND" H 4750 2980 30  0001 C CNN
 F 2 "" H 4750 3050 60  0000 C CNN
@@
 	4750 2900 4750 3050
 $Comp
-L +5V #PWR021
+L +5V #PWR20
 U 1 1 51E8266A
 P 7850 950
-F 0 "#PWR021" H 7850 1040 20  0001 C CNN
+F 0 "#PWR20" H 7850 1040 20  0001 C CNN
 F 1 "+5V" H 7850 1040 30  0000 C CNN
 F 2 "" H 7850 950 60  0000 C CNN
@@
 $EndComp
 $Comp
-L GND #PWR022
+L GND #PWR21
 U 1 1 51E8267F
 P 7850 2150
-F 0 "#PWR022" H 7850 2150 30  0001 C CNN
+F 0 "#PWR21" H 7850 2150 30  0001 C CNN
 F 1 "GND" H 7850 2080 30  0001 C CNN
 F 2 "" H 7850 2150 60  0000 C CNN
@@
 	7850 950  7850 1050
 $Comp
-L VDD #PWR023
+L VDD #PWR22
 U 1 1 51E827A2
 P 8200 950
-F 0 "#PWR023" H 8200 1050 30  0001 C CNN
+F 0 "#PWR22" H 8200 1050 30  0001 C CNN
 F 1 "VDD" H 8200 1060 30  0000 C CNN
 F 2 "" H 8200 950 60  0000 C CNN
@@
 	8200 1550 8200 1650
 $Comp
-L GND #PWR024
+L GND #PWR23
 U 1 1 51E82857
 P 8200 2150
-F 0 "#PWR024" H 8200 2150 30  0001 C CNN
+F 0 "#PWR23" H 8200 2150 30  0001 C CNN
 F 1 "GND" H 8200 2080 30  0001 C CNN
 F 2 "" H 8200 2150 60  0000 C CNN
@@
 	8200 2050 8200 2150
 $Comp
-L GND #PWR025
+L GND #PWR25
 U 1 1 51E828BA
 P 9000 950
-F 0 "#PWR025" H 9000 950 30  0001 C CNN
+F 0 "#PWR25" H 9000 950 30  0001 C CNN
 F 1 "GND" H 9000 880 30  0001 C CNN
 F 2 "" H 9000 950 60  0000 C CNN
@@
 	8750 1550 8750 1650
 $Comp
-L VSS #PWR026
+L VSS #PWR24
 U 1 1 51E829CC
 P 8750 2150
-F 0 "#PWR026" H 8750 2150 30  0001 C CNN
+F 0 "#PWR24" H 8750 2150 30  0001 C CNN
 F 1 "VSS" H 8750 2080 30  0000 C CNN
 F 2 "" H 8750 2150 60  0000 C CNN
@@
 Wire Wire Line
 	8450 2050 8200 2050
+$Comp
+L CONN_1 P1
+U 1 1 51E82EE8
+P 7900 2900
+F 0 "P1" H 7980 2900 40  0000 L CNN
+F 1 "V+" H 7900 2955 30  0001 C CNN
+F 2 "" H 7900 2900 60  0000 C CNN
+F 3 "" H 7900 2900 60  0000 C CNN
+	1    7900 2900
+	1    0    0    -1
+$EndComp
+$Comp
+L CONN_1 P2
+U 1 1 51E82EF5
+P 7900 3000
+F 0 "P2" H 7980 3000 40  0000 L CNN
+F 1 "GND" H 7900 3055 30  0001 C CNN
+F 2 "" H 7900 3000 60  0000 C CNN
+F 3 "" H 7900 3000 60  0000 C CNN
+	1    7900 3000
+	1    0    0    -1
+$EndComp
+$Comp
+L CONN_1 P3
+U 1 1 51E82EFB
+P 7900 3100
+F 0 "P3" H 7980 3100 40  0000 L CNN
+F 1 "V-" H 7900 3155 30  0001 C CNN
+F 2 "" H 7900 3100 60  0000 C CNN
+F 3 "" H 7900 3100 60  0000 C CNN
+	1    7900 3100
+	1    0    0    -1
+$EndComp
+$Comp
+L CONN_1 P4
+U 1 1 51E82F0B
+P 7600 4550
+F 0 "P4" H 7680 4550 40  0000 L CNN
+F 1 "Out" H 7600 4605 30  0001 C CNN
+F 2 "" H 7600 4550 60  0000 C CNN
+F 3 "" H 7600 4550 60  0000 C CNN
+	1    7600 4550
+	1    0    0    -1
+$EndComp
+$Comp
+L CONN_1 P5
+U 1 1 51E82F11
+P 7600 4750
+F 0 "P5" H 7680 4750 40  0000 L CNN
+F 1 "GND" H 7600 4805 30  0001 C CNN
+F 2 "" H 7600 4750 60  0000 C CNN
+F 3 "" H 7600 4750 60  0000 C CNN
+	1    7600 4750
+	1    0    0    -1
+$EndComp
 $EndSCHEMATC
