File: dac_shield.sch (KiCad schematic (older format))
At the start: 27 parts, among them P1 CONN_2, P2 CONN_2, P3 CONN_2, T1 VrefTest, U1 MCP4921, U2 TCA0372, U3 LM741

Commit message: Changed to 2017
Parts:
- C1, C2, C3, C4: symbol C -> C-RESCUE-dac_shield
- D1, D2, D3: symbol LED -> LED-RESCUE-dac_shield
- R1, R2, R3, R4, R5, R6, R7, R8, R9: symbol R -> R-RESCUE-dac_shield
- U3: symbol LM741 -> LM741-RESCUE-dac_shield
Changed lines of the file:
@@
 EESchema Schematic File Version 2
+LIBS:dac_shield-rescue
 LIBS:power
 LIBS:device
@@
 LIBS:custom_parts
 LIBS:dac_shield-cache
-EELAYER 27 0
+EELAYER 25 0
 EELAYER END
 $Descr USLetter 11000 8500
@@
 	5200 2100 5200 1950
 $Comp
-L GND #PWR03
+L GND-RESCUE-dac_shield #PWR03
 U 1 1 51E30124
 P 3900 1550
@@
 	3900 1450 3900 1550
 $Comp
-L GND #PWR04
+L GND-RESCUE-dac_shield #PWR04
 U 1 1 51E3017A
 P 1150 2200
@@
 $EndComp
 $Comp
-L GND #PWR05
+L GND-RESCUE-dac_shield #PWR05
 U 1 1 51E30180
 P 6350 2300
@@
 	5350 4450 5650 4450
 $Comp
-L R R4
+L R-RESCUE-dac_shield R4
 U 1 1 51E30590
 P 4650 5150
@@
 	5650 5050 5650 4650
 $Comp
-L R R6
+L R-RESCUE-dac_shield R6
 U 1 1 51E30757
 P 6300 5200
@@
 	6550 5200 6550 4550
 $Comp
-L R R5
+L R-RESCUE-dac_shield R5
 U 1 1 51E307BD
 P 5300 5550
@@
 	5300 5200 5400 5200
 $Comp
-L GND #PWR010
+L GND-RESCUE-dac_shield #PWR010
 U 1 1 51E307ED
 P 5300 5950
@@
 	5300 5800 5300 5950
 $Comp
-L R R3
+L R-RESCUE-dac_shield R3
 U 1 1 51E3081F
 P 3900 4650
@@
 DAC_OUT
 $Comp
-L LM741 U3
+L LM741-RESCUE-dac_shield U3
 U 1 1 51E30A12
 P 2100 4650
@@
 	2000 4150 2000 4250
 $Comp
-L R R1
+L R-RESCUE-dac_shield R1
 U 1 1 51E30B0D
 P 1400 4300
@@
 $EndComp
 $Comp
-L R R2
+L R-RESCUE-dac_shield R2
 U 1 1 51E30B19
 P 1400 4900
@@
 $EndComp
 $Comp
-L GND #PWR014
+L GND-RESCUE-dac_shield #PWR014
 U 1 1 51E30B25
 P 1400 5250
@@
 	7500 3100 7500 3250
 $Comp
-L GND #PWR017
+L GND-RESCUE-dac_shield #PWR017
 U 1 1 51E30E0E
 P 7350 3050
@@
 Connection ~ 6550 4550
 $Comp
-L GND #PWR018
+L GND-RESCUE-dac_shield #PWR018
 U 1 1 51E30EF3
 P 7300 4850
@@
 	7300 4750 7450 4750
 $Comp
-L C C1
+L C-RESCUE-dac_shield C1
 U 1 1 51E82508
 P 1050 4900
@@
 	1050 5150 1400 5150
 $Comp
-L C C2
+L C-RESCUE-dac_shield C2
 U 1 1 51E825BA
 P 4750 2700
@@
 Connection ~ 5200 2100
 $Comp
-L GND #PWR019
+L GND-RESCUE-dac_shield #PWR019
 U 1 1 51E82617
 P 4750 3050
@@
 $EndComp
 $Comp
-L LED D1
+L LED-RESCUE-dac_shield D1
 U 1 1 51E82672
 P 7850 1850
@@
 $EndComp
 $Comp
-L GND #PWR021
+L GND-RESCUE-dac_shield #PWR021
 U 1 1 51E8267F
 P 7850 2150
@@
 $EndComp
 $Comp
-L R R7
+L R-RESCUE-dac_shield R7
 U 1 1 51E8268F
 P 7850 1300
@@
 $EndComp
 $Comp
-L R R8
+L R-RESCUE-dac_shield R8
 U 1 1 51E827A8
 P 8200 1300
@@
 	8200 950  8200 1050
 $Comp
-L LED D2
+L LED-RESCUE-dac_shield D2
 U 1 1 51E827FF
 P 8200 1850
@@
 	8200 1550 8200 1650
 $Comp
-L GND #PWR023
+L GND-RESCUE-dac_shield #PWR023
 U 1 1 51E82857
 P 8200 2150
@@
 	8200 2050 8200 2150
 $Comp
-L GND #PWR024
+L GND-RESCUE-dac_shield #PWR024
 U 1 1 51E828BA
 P 9000 950
@@
 $EndComp
 $Comp
-L R R9
+L R-RESCUE-dac_shield R9
 U 1 1 51E82914
 P 8750 1300
@@
 	9000 850  9000 950
 $Comp
-L LED D3
+L LED-RESCUE-dac_shield D3
 U 1 1 51E8296F
 P 8750 1850
@@
 	7850 2050 7850 2150
 $Comp
-L C C4
+L C-RESCUE-dac_shield C4
 U 1 1 51E82BF5
 P 9100 1600
@@
 	9100 2050 9100 1800
 $Comp
-L C C3
+L C-RESCUE-dac_shield C3
 U 1 1 51E82CAF
 P 8450 1600
@@
 	8450 2050 8200 2050
 $Comp
-L GND #PWR026
+L GND-RESCUE-dac_shield #PWR026
 U 1 1 51EEC648
 P 6250 2700
